Commit message: changes

File: line_following/models/line_following_robot/robot.urdf (robot description, URDF)
Before this commit: robot line_follower_robot, 4 links, 3 joints
Links:
- link base_link: geometry collision mesh filename=model://line_following_robot/waffle_pi_base.dae scale=1 1 1; visual mesh filename=model://line_following_robot/waffle_pi_base.dae scale=1 1 1
- link left_wheel: geometry collision mesh filename=model://line_following_robot/tire.dae scale=1 1 1; visual mesh filename=model://line_following_robot/tire.dae scale=1 1 1
- link right_wheel: geometry collision mesh filename=model://line_following_robot/tire.dae scale=1 1 1; visual mesh filename=model://line_following_robot/tire.dae scale=1 1 1
